Commit message: fix : visual joint states work

File: src/robot_moveit_config_tb/config/armr5.ros2_control.xacro (robot description, xacro)
@@ -5,6 +5,5 @@
         <ros2_control name="${name}" type="system">
             <hardware>
-                <!-- By default, set up controllers for simulation. This won't work on real hardware -->
-                <plugin>mock_components/GenericSystem</plugin>
+                <plugin>robot_hardware_interface/SlushEngineHardware</plugin>
             </hardware>
             <joint name="R0_Yaw">
@@ -50,39 +49,4 @@
                 <state_interface name="velocity"/>
             </joint>
-            <joint name="LeftGripper">
-                <command_interface name="position"/>
-                <state_interface name="position">
-                  <param name="initial_value">${initial_positions['LeftGripper']}</param>
-                </state_interface>
-                <state_interface name="velocity"/>
-            </joint>
-            <joint name="LeftPivotArm">
-                <command_interface name="position"/>
-                <state_interface name="position">
-                  <param name="initial_value">${initial_positions['LeftPivotArm']}</param>
-                </state_interface>
-                <state_interface name="velocity"/>
-            </joint>
-            <joint name="PassifGear">
-                <command_interface name="position"/>
-                <state_interface name="position">
-                  <param name="initial_value">${initial_positions['PassifGear']}</param>
-                </state_interface>
-                <state_ interface name="velocity"/>
-            </joint>
-            <joint name="RightGripper">
-                <command_interface name="position"/>
-                <state_interface name="position">
-                  <param name="initial_value">${initial_positions['RightGripper']}</param>
-                </state_interface>
-                <state_interface name="velocity"/>
-            </joint>
-            <joint name="RightPivotArm">
-                <command_interface name="position"/>
-                <state_interface name="position">
-                  <param name="initial_value">${initial_positions['RightPivotArm']}</param>
-                </state_interface>
-                <state_interface name="velocity"/>
-            </joint>
         </ros2_control>
     </xacro:macro>
