Commit message: fix : launch can be started but stuck

File: src/robot_description_tb/urdf/r5a_v_ros.urdf.xacro (robot description, xacro)
@@ -336,5 +336,4 @@
       effort="5"
       velocity="1" />
-  </joint>
   </joint>
   <link
@@ -710,5 +709,4 @@
       <state_interface name="position" />
     </joint>
-  </ros2_control>
     <joint name="ServoGear">
       <command_interface name="position"/>
@@ -718,3 +716,4 @@
       <state_interface name="velocity"/>
     </joint>
+    </ros2_control>
 </robot>

Commit message: fix : everything start

File: src/robot_description_tb/urdf/r5a_v_ros.urdf.xacro (robot description, xacro)
@@ -686,34 +686,37 @@
   </joint>
   <ros2_control name="TBRobotSystem" type="system">
-    <hardware>
-      <plugin>robot_hardware_interface/SlushEngineHardware</plugin>
-    </hardware>
-    <joint name="R0_Yaw">
-      <command_interface name="position" />
-      <state_interface name="position" />
-    </joint>
-    <joint name="R1_Pitch">
-      <command_interface name="position" />
-      <state_interface name="position" />
-    </joint>
-    <joint name="R2_Pitch">
-      <command_interface name="position" />
-      <state_interface name="position" />
-    </joint>
-    <joint name="R3_Yaw">
-      <command_interface name="position" />
-      <state_interface name="position" />
-    </joint>
-    <joint name="R4_Pitch">
-      <command_interface name="position" />
-      <state_interface name="position" />
-    </joint>
-    <joint name="ServoGear">
-      <command_interface name="position"/>
-      <state_interface name="position">
-        <param name="initial_value">0.0</param>
-      </state_interface>
-      <state_interface name="velocity"/>
-    </joint>
-    </ros2_control>
+      <hardware>
+          <plugin>robot_hardware_interface/SlushEngineHardware</plugin>
+      </hardware>
+      <joint name="R0_Yaw">
+          <command_interface name="position"/>
+          <state_interface name="position"/>
+          <state_interface name="velocity"/>
+      </joint>
+      <joint name="R1_Pitch">
+          <command_interface name="position"/>
+          <state_interface name="position"/>
+          <state_interface name="velocity"/>
+      </joint>
+      <joint name="R2_Pitch">
+          <command_interface name="position"/>
+          <state_interface name="position"/>
+          <state_interface name="velocity"/>
+      </joint>
+      <joint name="R3_Yaw">
+          <command_interface name="position"/>
+          <state_interface name="position"/>
+          <state_interface name="velocity"/>
+      </joint>
+      <joint name="R4_Pitch">
+          <command_interface name="position"/>
+          <state_interface name="position"/>
+          <state_interface name="velocity"/>
+      </joint>
+      <joint name="ServoGear">
+          <command_interface name="position"/>
+          <state_interface name="position"/>
+          <state_interface name="velocity"/>
+      </joint>
+  </ros2_control>
 </robot>

Commit message: fix: make moveit not expect the passifs joints

File: src/robot_description_tb/urdf/r5a_v_ros.urdf.xacro (robot description, xacro)
@@ -685,38 +685,50 @@
       velocity="1" />
   </joint>
-  <ros2_control name="TBRobotSystem" type="system">
-      <hardware>
-          <plugin>robot_hardware_interface/SlushEngineHardware</plugin>
-      </hardware>
-      <joint name="R0_Yaw">
-          <command_interface name="position"/>
-          <state_interface name="position"/>
-          <state_interface name="velocity"/>
-      </joint>
-      <joint name="R1_Pitch">
-          <command_interface name="position"/>
-          <state_interface name="position"/>
-          <state_interface name="velocity"/>
-      </joint>
-      <joint name="R2_Pitch">
-          <command_interface name="position"/>
-          <state_interface name="position"/>
-          <state_interface name="velocity"/>
-      </joint>
-      <joint name="R3_Yaw">
-          <command_interface name="position"/>
-          <state_interface name="position"/>
-          <state_interface name="velocity"/>
-      </joint>
-      <joint name="R4_Pitch">
-          <command_interface name="position"/>
-          <state_interface name="position"/>
-          <state_interface name="velocity"/>
-      </joint>
-      <joint name="ServoGear">
-          <command_interface name="position"/>
-          <state_interface name="position"/>
-          <state_interface name="velocity"/>
-      </joint>
-  </ros2_control>
+<ros2_control name="TBRobotSystem" type="system">
+            <hardware>
+                <plugin>robot_hardware_interface/SlushEngineHardware</plugin>
+            </hardware>
+            <joint name="R0_Yaw">
+                <param name="id">0</param>
+                <command_interface name="position"/>
+                <state_interface name="position">
+                </state_interface>
+                <state_interface name="velocity"/>
+            </joint>
+            <joint name="R1_Pitch">
+                <param name="id">1</param>
+                <command_interface name="position"/>
+                <state_interface name="position">
+                </state_interface>
+                <state_interface name="velocity"/>
+            </joint>
+            <joint name="R2_Pitch">
+                <param name="id">2</param>
+                <command_interface name="position"/>
+                <state_interface name="position">
+                </state_interface>
+                <state_interface name="velocity"/>
+            </joint>
+            <joint name="R3_Yaw">
+                <param name="id">3</param>
+                <command_interface name="position"/>
+                <state_interface name="position">
+                </state_interface>
+                <state_interface name="velocity"/>
+            </joint>
+            <joint name="R4_Pitch">
+                <param name="id">4</param>
+                <command_interface name="position"/>
+                <state_interface name="position">
+                </state_interface>
+                <state_interface name="velocity"/>
+            </joint>
+            <joint name="ServoGear">
+                <param name="id">5</param>
+                <command_interface name="position"/>
+                <state_interface name="position">
+                </state_interface>
+                <state_interface name="velocity"/>
+            </joint>
+        </ros2_control>
 </robot>

File: src/robot_moveit_config_tb/config/armr5.ros2_control.xacro (robot description, xacro)
@@ -8,42 +8,48 @@
             </hardware>
             <joint name="R0_Yaw">
+                <param name="id">0</param>
                 <command_interface name="position"/>
                 <state_interface name="position">
-                  <param name="initial_value">${initial_positions['R0_Yaw']}</param>
+                    <param name="initial_value">${initial_positions['R0_Yaw']}</param>
                 </state_interface>
                 <state_interface name="velocity"/>
             </joint>
             <joint name="R1_Pitch">
+                <param name="id">1</param>
                 <command_interface name="position"/>
                 <state_interface name="position">
-                  <param name="initial_value">${initial_positions['R1_Pitch']}</param>
+                    <param name="initial_value">${initial_positions['R1_Pitch']}</param>
                 </state_interface>
                 <state_interface name="velocity"/>
             </joint>
             <joint name="R2_Pitch">
+                <param name="id">2</param>
                 <command_interface name="position"/>
                 <state_interface name="position">
-                  <param name="initial_value">${initial_positions['R2_Pitch']}</param>
+                    <param name="initial_value">${initial_positions['R2_Pitch']}</param>
                 </state_interface>
                 <state_interface name="velocity"/>
             </joint>
             <joint name="R3_Yaw">
+                <param name="id">3</param>
                 <command_interface name="position"/>
                 <state_interface name="position">
-                  <param name="initial_value">${initial_positions['R3_Yaw']}</param>
+                    <param name="initial_value">${initial_positions['R3_Yaw']}</param>
                 </state_interface>
                 <state_interface name="velocity"/>
             </joint>
             <joint name="R4_Pitch">
+                <param name="id">4</param>
                 <command_interface name="position"/>
                 <state_interface name="position">
-                  <param name="initial_value">${initial_positions['R4_Pitch']}</param>
+                    <param name="initial_value">${initial_positions['R4_Pitch']}</param>
                 </state_interface>
                 <state_interface name="velocity"/>
             </joint>
             <joint name="ServoGear">
+                <param name="id">5</param>
                 <command_interface name="position"/>
                 <state_interface name="position">
-                  <param name="initial_value">${initial_positions['ServoGear']}</param>
+                    <param name="initial_value">${initial_positions['ServoGear']}</param>
                 </state_interface>
                 <state_interface name="velocity"/>

Commit message: fix: put mimic in urdf for the passif gripper joints

File: src/robot_description_tb/urdf/r5a_v_ros.urdf.xacro (robot description, xacro)
@@ -279,456 +279,247 @@
       velocity="1" />
   </joint>
-  <link
-    name="R5A_link5">
-    <inertial>
-      <origin
-        xyz="-0.000304982815722917 0.000214555031841958 0.0238812711123602"
-        rpy="0 0 0" />
-      <mass
-        value="0.232244400597819" />
-      <inertia
-        ixx="0.000120322215361587"
-        ixy="-9.01049257248474E-08"
-        ixz="2.57785604684289E-07"
-        iyy="9.55044143695027E-05"
-        iyz="-7.60482494086889E-08"
-        izz="6.98522198363616E-05" />
-    </inertial>
-    <visual>
-      <origin
-        xyz="0 0 0"
-        rpy="0 0 0" />
-      <geometry>
-        <mesh
-          filename="file://$(find robot_description_tb)/meshes/R5A_link5.STL" />
-      </geometry>
-      <material
-        name="">
-        <color
-          rgba="1 1 1 1" />
-      </material>
-    </visual>
-    <collision>
-      <origin
-        xyz="0 0 0"
-        rpy="0 0 0" />
-      <geometry>
-        <mesh
-          filename="file://$(find robot_description_tb)/meshes/R5A_link5.STL" />
-      </geometry>
-    </collision>
-  </link>
-  <joint
-    name="R4_Pitch"
-    type="revolute">
-    <origin
-      xyz="0 0.095 0"
-      rpy="1.5708 0 3.1416" />
-    <parent
-      link="R5A_link4" />
-    <child
-      link="R5A_link5" />
-    <axis
-      xyz="-1 0 0" />
-    <limit
-      lower="-1.5"
-      upper="1.5"
-      effort="5"
-      velocity="1" />
-  </joint>
-  <link
-    name="R5A_GripperLeft_Link1">
-    <inertial>
-      <origin
-        xyz="-0.00659452357779758 -0.000394229793377554 2.33412007890428E-06"
-        rpy="0 0 0" />
-      <mass
-        value="0.00487858122952023" />
-      <inertia
-        ixx="2.28094324920978E-07"
-        ixy="1.69392169643129E-08"
-        ixz="-1.00081436396101E-10"
-        iyy="9.51062234425361E-07"
-        iyz="1.21242073786193E-09"
-        izz="1.15060635431209E-06" />
-    </inertial>
-    <visual>
-      <origin
-        xyz="0 0 0"
-        rpy="0 0 0" />
-      <geometry>
-        <mesh
-          filename="file://$(find robot_description_tb)/meshes/R5A_GripperLeft_Link1.STL" />
-      </geometry>
-      <material
-        name="">
-        <color
-          rgba="1 1 1 1" />
-      </material>
-    </visual>
-    <collision>
-      <origin
-        xyz="0 0 0"
-        rpy="0 0 0" />
-      <geometry>
-        <mesh
-          filename="file://$(find robot_description_tb)/meshes/R5A_GripperLeft_Link1.STL" />
-      </geometry>
-    </collision>
-  </link>
-  <joint
-    name="ServoGear"
-    type="revolute">
-    <origin
-      xyz="0.0140000000000435 -0.000394292596204153 0.0649988040916903"
-      rpy="1.5707963267949 0 3.14159265358979" />
-    <parent
-      link="R5A_link5" />
-    <child
-      link="R5A_GripperLeft_Link1" />
-    <axis
-      xyz="0 -0.006066039941515 -0.99998160141046" />
-    <limit
-      lower="-0.01"
-      upper="1.0"
-      effort="5"
-      velocity="1" />
-  </joint>
-  <link
-    name="R5A_GripperLeft_Link2">
-    <inertial>
-      <origin
-        xyz="0.0121769148397674 0.0264987914633908 -0.00015844305881356"
-        rpy="0 0 0" />
-      <mass
-        value="0.010285119366326" />
-      <inertia
-        ixx="3.24436687710476E-06"
-        ixy="-1.54511287979719E-06"
-        ixz="9.58011795509873E-09"
-        iyy="1.30527398272079E-06"
-        iyz="1.62739383329718E-08"
-        izz="3.9267289910886E-06" />
-    </inertial>
-    <visual>
-      <origin
-        xyz="0 0 0"
-        rpy="0 0 0" />
-      <geometry>
-        <mesh
-          filename="file://$(find robot_description_tb)/meshes/R5A_GripperLeft_Link2.STL" />
-      </geometry>
-      <material
-        name="">
-        <color
-          rgba="0.792156862745098 0.819607843137255 0.933333333333333 1" />
-      </material>
-    </visual>
-    <collision>
-      <origin
-        xyz="0 0 0"
-        rpy="0 0 0" />
-      <geometry>
-        <mesh
-          filename="file://$(find robot_description_tb)/meshes/R5A_GripperLeft_Link2.STL" />
-      </geometry>
-    </collision>
-  </link>
-  <joint
-    name="LeftGripper"
-    type="revolute">
-    <origin
-      xyz="-0.0399999995050676 0 0"
-      rpy="0 0 0" />
-    <parent
-      link="R5A_GripperLeft_Link1" />
-    <child
-      link="R5A_GripperLeft_Link2" />
-    <axis
-      xyz="0 -0.00606603994152109 -0.99998160141046" />
-    <limit
-      lower="-1.0"
-      upper="0.01"
-      effort="5"
-      velocity="1" />
-  </joint>
-  <link
-    name="R5A_GripperRight_Link1">
-    <inertial>
-      <origin
-        xyz="0.00645173751362635 -0.000420742089632498 2.55112204775943E-06"
-        rpy="0 0 0" />
-      <mass
-        value="0.0050032197309173" />
-      <inertia
-        ixx="2.29355330577406E-07"
-        ixy="-1.79692415236652E-08"
-        ixz="1.09050530560748E-10"
-        iyy="9.5760807063583E-07"
-        iyz="1.21374586203625E-09"
-        izz="1.15767989130762E-06" />
-    </inertial>
-    <visual>
-      <origin
-        xyz="0 0 0"
-        rpy="0 0 0" />
-      <geometry>
-        <mesh
-          filename="file://$(find robot_description_tb)/meshes/R5A_GripperRight_Link1.STL" />
-      </geometry>
-      <material
-        name="">
-        <color
-          rgba="1 1 1 1" />
-      </material>
-    </visual>
-    <collision>
-      <origin
-        xyz="0 0 0"
-        rpy="0 0 0" />
-      <geometry>
-        <mesh
-          filename="file://$(find robot_description_tb)/meshes/R5A_GripperRight_Link1.STL" />
-      </geometry>
-    </collision>
-  </link>
-  <joint
-    name="PassifGear"
-    type="revolute">
-    <origin
-      xyz="-0.014 -0.00039429 0.064999"
-      rpy="1.5708 0 3.1416" />
-    <parent
-      link="R5A_link5" />
-    <child
-      link="R5A_GripperRight_Link1" />
-    <axis
-      xyz="0 -0.006066 -0.99998" />
-    <limit
-      lower="-1.0"
-      upper="0.01"
-      effort="5"
-      velocity="1" />
-  </joint>
-  <link
-    name="R5A_GripperRight_Link2">
-    <inertial>
-      <origin
-        xyz="-0.0121769121022437 0.0264987629997102 -0.000158239935641401"
-        rpy="0 0 0" />
-      <mass
-        value="0.010285143205825" />
-      <inertia
-        ixx="3.24437190589205E-06"
-        ixy="1.54511360510839E-06"
-        ixz="-9.56821825775037E-09"
-        iyy="1.30527511012569E-06"
-        iyz="1.63061443850165E-08"
-        izz="3.92673308798733E-06" />
-    </inertial>
-    <visual>
-      <origin
-        xyz="0 0 0"
-        rpy="0 0 0" />
-      <geometry>
-        <mesh
-          filename="file://$(find robot_description_tb)/meshes/R5A_GripperRight_Link2.STL" />
-      </geometry>
-      <material
-        name="">
-        <color
-          rgba="0.792156862745098 0.819607843137255 0.933333333333333 1" />
-      </material>
-    </visual>
-    <collision>
-      <origin
-        xyz="0 0 0"
-        rpy="0 0 0" />
-      <geometry>
-        <mesh
-          filename="file://$(find robot_description_tb)/meshes/R5A_GripperRight_Link2.STL" />
-      </geometry>
-    </collision>
-  </link>
-  <joint
-    name="RightGripper"
-    type="revolute">
-    <origin
-      xyz="0.0399999045264166 -8.73933436228436E-05 0"
-      rpy="0 0 0" />
-    <parent
-      link="R5A_GripperRight_Link1" />
-    <child
-      link="R5A_GripperRight_Link2" />
-    <axis
-      xyz="0 -0.00606603994152205 -0.99998160141046" />
-    <limit
-      lower="-0.01"
-      upper="1.0"
-      effort="5"
-      velocity="1" />
-  </joint>
-  <link
-    name="R5A_GripperLeft_Link3">
-    <inertial>
-      <origin
-        xyz="-0.0199999997525652 3.14595219752523E-06 -1.9083866895607E-08"
-        rpy="0 0 0" />
-      <mass
-        value="0.00167027391699932" />
-      <inertia
-        ixx="1.0506836483145E-08"
-        ixy="4.70838754646716E-11"
-        ixz="-2.85618585168146E-13"
-        iyy="3.09836744743029E-07"
-        iyz="5.57882383972831E-12"
-        izz="3.10756375336318E-07" />
-    </inertial>
-    <visual>
-      <origin
-        xyz="0 0 0"
-        rpy="0 0 0" />
-      <geometry>
-        <mesh
-          filename="file://$(find robot_description_tb)/meshes/R5A_GripperLeft_Link3.STL" />
-      </geometry>
-      <material
-        name="">
-        <color
-          rgba="1 1 1 1" />
-      </material>
-    </visual>
-    <collision>
-      <origin
-        xyz="0 0 0"
-        rpy="0 0 0" />
-      <geometry>
-        <mesh
-          filename="file://$(find robot_description_tb)/meshes/R5A_GripperLeft_Link3.STL" />
-      </geometry>
-    </collision>
-  </link>
-  <joint
-    name="LeftPivotArm"
-    type="revolute">
-    <origin
-      xyz="0.007000000000237 -0.000515613395019377 0.0849984361199003"
-      rpy="1.5707963267949 0 3.14159265358979" />
-    <parent
-      link="R5A_link5" />
-    <child
-      link="R5A_GripperLeft_Link3" />
-    <axis
-      xyz="0 0.00606603994152107 0.99998160141046" />
-    <limit
-      lower="-1.0"
-      upper="0.01"
-      effort="5"
-      velocity="1" />
-  </joint>
-  <link
-    name="R5A_GripperRight_Link3">
-    <inertial>
-      <origin
-        xyz="0.0199999522633234 -4.36966718082576E-05 2.65070677277451E-07"
-        rpy="0 0 0" />
-      <mass
-        value="0.00167027391699932" />
-      <inertia
-        ixx="1.05082579798437E-08"
-        ixy="6.53984435711288E-10"
-        ixz="-3.96716935937682E-12"
-        iyy="3.09835323298637E-07"
-        iyz="5.58744653817654E-12"
-        izz="3.10756375284011E-07" />
-    </inertial>
-    <visual>
-      <origin
-        xyz="0 0 0"
-        rpy="0 0 0" />
-      <geometry>
-        <mesh
-          filename="file://$(find robot_description_tb)/meshes/R5A_GripperRight_Link3.STL" />
-      </geometry>
-      <material
-        name="">
-        <color
-          rgba="1 1 1 1" />
-      </material>
-    </visual>
-    <collision>
-      <origin
-        xyz="0 0 0"
-        rpy="0 0 0" />
-      <geometry>
-        <mesh
-          filename="file://$(find robot_description_tb)/meshes/R5A_GripperRight_Link3.STL" />
-      </geometry>
-    </collision>
-  </link>
-  <joint
-    name="RightPivotArm"
-    type="revolute">
-    <origin
-      xyz="-0.00699999999995929 -0.000515613394988563 0.0849984361199004"
-      rpy="1.5707963267949 0 3.14159265358979" />
-    <parent
-      link="R5A_link5" />
-    <child
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